File: src/Rs485IsoFEC.kicad_pcb (KiCad board)
At the start: 2 copper layers, 24 x 27.9 mm, 27 parts, among them J1 B4B-XH-A, P1 105444-0001, Q1 DMP3099L-13, U1 FT232RL, U2 ADM2682E

Commit message: Moved termination resistor
Parts:
- moved R1 5.30 mm to (37.3, 37.9), turned to 180 degrees
Routing:
- net ISO_A: track 26.8 -> 24.3 mm
- net ISO_GND: track 32.0 -> 30.6 mm
- net ISO_B: track 24.3 -> 23.0 mm
Changed lines of the file:
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@@
   )
   (footprint "Medo64:R (0805)" (layer "F.Cu")
-    (at 32 37.85)
+    (at 37.3 37.85 180)
     (tags "RESC2013X70N")
     (attr smd)
@@
         (effects (font (size 0.8 0.6) (thickness 0.15)))
     )
-    (fp_text value "TERM" (at 0 -1.45) (layer "F.SilkS")
+    (fp_text value "TERM" (at -0.7 -1.55 180) (layer "F.SilkS")
         (effects (font (size 0.8 0.6) (thickness 0.15)))
     )
@@
     (fp_rect (start -1 -0.625) (end 1 0.625)
       (stroke (width 0.01) (type dash_dot)) (fill none) (layer "F.Fab"))
-    (pad "1" smd roundrect (at -0.95 0) (size 1.05 1.4) (layers "F.Cu" "F.Paste" "F.Mask") (roundrect_rratio 0.25)
+    (pad "1" smd roundrect (at -0.95 0 180) (size 1.05 1.4) (layers "F.Cu" "F.Paste" "F.Mask") (roundrect_rratio 0.25)
       (net 21 "ISO_A") (thermal_bridge_angle 45))
-    (pad "2" smd roundrect (at 0.95 0) (size 1.05 1.4) (layers "F.Cu" "F.Paste" "F.Mask") (roundrect_rratio 0.25)
+    (pad "2" smd roundrect (at 0.95 0 180) (size 1.05 1.4) (layers "F.Cu" "F.Paste" "F.Mask") (roundrect_rratio 0.25)
       (net 22 "ISO_B") (thermal_bridge_angle 45))
     (model ":KICAD7_3DMODEL_DIR:Resistor_SMD.3dshapes/R_0805_2012Metric.step"
@@
     (effects (font (size 0.8 0.6) (thickness 0.15) bold) (justify mirror))
   )
-  (gr_text "GND" (at 28.2 38.6) (layer "F.SilkS" knockout)
+  (gr_text "GND" (at 28.2 38.7) (layer "F.SilkS" knockout)
     (effects (font (size 1.3 0.9) (thickness 0.15) bold) (justify bottom))
   )
-  (gr_text "B" (at 34.5 40.8) (layer "F.SilkS" knockout)
+  (gr_text "B" (at 33.2 38.7) (layer "F.SilkS" knockout)
     (effects (font (size 1.3 0.9) (thickness 0.15) bold) (justify bottom))
   )
-  (gr_text "A" (at 32 40.8) (layer "F.SilkS" knockout)
+  (gr_text "A" (at 30.8 38.7) (layer "F.SilkS" knockout)
     (effects (font (size 1.3 0.9) (thickness 0.15) bold) (justify bottom))
   )
@@
   (segment (start 38.799659 42.399659) (end 25.300341 42.399659) (width 0.2) (layer "B.Cu") (net 3))
   (segment (start 25.300341 42.399659) (end 25 42.7) (width 0.2) (layer "B.Cu") (net 3))
-  (segment (start 22.75 44) (end 22.75 44.1) (width 0.2) (layer "B.Cu") (net 3))
   (segment (start 24.05 42.7) (end 22.75 44) (width 0.2) (layer "B.Cu") (net 3))
   (segment (start 26.7 29.4) (end 25.6 29.4) (width 0.2) (layer "B.Cu") (net 3))
@@
   (segment (start 38.805026 41.8) (end 24.7 41.8) (width 0.2) (layer "B.Cu") (net 10))
   (segment (start 41.35 44.1) (end 41.35 46.45) (width 0.2) (layer "B.Cu") (net 11))
-  (segment (start 41.35 46.45) (end 41.3 46.5) (width 0.2) (layer "B.Cu") (net 11))
-  (segment (start 24.5 44.25) (end 24.65 44.1) (width 0.2) (layer "B.Cu") (net 12))
   (segment (start 24.5 46.5) (end 24.5 44.25) (width 0.2) (layer "B.Cu") (net 12))
   (segment (start 22.1 30.325) (end 23.525 30.325) (width 0.2) (layer "F.Cu") (net 13))
@@
   (segment (start 35.3 33) (end 37.5 33) (width 0.2) (layer "B.Cu") (net 14))
   (segment (start 30.325 34.2) (end 31.075 33.45) (width 0.2) (layer "B.Cu") (net 14))
-  (segment (start 32.65 33.2) (end 32.4 33.45) (width 0.2) (layer "B.Cu") (net 14))
   (segment (start 28.3 34.2) (end 30.325 34.2) (width 0.2) (layer "B.Cu") (net 14))
   (segment (start 29.45 31.4) (end 27.3 31.4) (width 0.2) (layer "B.Cu") (net 15))
@@
   (segment (start 27.1 28.294974) (end 27.669974 27.725) (width 0.2) (layer "F.Cu") (net 18))
   (segment (start 26.85 29.75) (end 27.1 29.5) (width 0.2) (layer "F.Cu") (net 18))
-  (segment (start 28.25 39.65) (end 28.25 40.8) (width 0.6) (layer "F.Cu") (net 19))
   (segment (start 41.045 25.755) (end 41 25.8) (width 0.2) (layer "F.Cu") (net 19))
   (segment (start 41.045 25.655) (end 40.9 25.8) (width 0.2) (layer "F.Cu") (net 19))
@@
   (via (at 40.9 34.5) (size 0.6) (drill 0.3) (layers "F.Cu" "B.Cu") (net 19))
   (via (at 28.25 39.65) (size 0.6) (drill 0.3) (layers "F.Cu" "B.Cu") (net 19))
-  (segment (start 39.9 26.2) (end 39.7 26.2) (width 0.2) (layer "B.Cu") (net 19))
   (segment (start 40.9 25.7) (end 41 25.8) (width 0.2) (layer "B.Cu") (net 19))
   (segment (start 28.25 39.65) (end 29.599998 38.300002) (width 0.6) (layer "B.Cu") (net 19))
@@
   (segment (start 32 37.4) (end 32.3 37.1) (width 0.3) (layer "B.Cu") (net 19))
   (segment (start 39.6 37.1) (end 39.9 36.8) (width 0.3) (layer "B.Cu") (net 19))
-  (segment (start 39.8 34.8) (end 39.9 34.8) (width 0.2) (layer "B.Cu") (net 19))
   (segment (start 39.9 36.8) (end 39.9 34.9) (width 0.3) (layer "B.Cu") (net 19))
   (segment (start 41 25.8) (end 41.7 25.8) (width 0.2) (layer "B.Cu") (net 19))
@@
   (segment (start 40.9 33.2) (end 41.9 33.2) (width 0.2) (layer "B.Cu") (net 20))
   (segment (start 40.8 27.6) (end 40.3 27.6) (width 0.2) (layer "B.Cu") (net 20))
-  (segment (start 31.05 37.7) (end 31.05 40.50001) (width 0.2) (layer "F.Cu") (net 21))
-  (segment (start 42.2 32.105) (end 40.695 32.105) (width 0.2) (layer "F.Cu") (net 21))
-  (segment (start 42.2 32.105) (end 43.095 32.105) (width 0.2) (layer "F.Cu") (net 21))
-  (segment (start 38.2 34.6) (end 38.2 38.6) (width 0.2) (layer "F.Cu") (net 21))
-  (segment (start 43.4 31.8) (end 43.4 28.6) (width 0.2) (layer "F.Cu") (net 21))
-  (segment (start 43.4 28.6) (end 43.095 28.295) (width 0.2) (layer "F.Cu") (net 21))
-  (segment (start 43.095 32.105) (end 43.4 31.8) (width 0.2) (layer "F.Cu") (net 21))
-  (segment (start 43.095 28.295) (end 42.2 28.295) (width 0.2) (layer "F.Cu") (net 21))
+  (segment (start 43.095 32.105) (end 40.695 32.105) (width 0.2) (layer "F.Cu") (net 21))
   (segment (start 40.695 32.105) (end 38.2 34.6) (width 0.2) (layer "F.Cu") (net 21))
-  (segment (start 31.05 41) (end 30.95 41) (width 0.5) (layer "F.Cu") (net 21))
-  (segment (start 30.95 41) (end 30.75 40.8) (width 0.5) (layer "F.Cu") (net 21))
-  (via (at 38.2 38.6) (size 0.6) (drill 0.3) (layers "F.Cu" "B.Cu") (net 21))
+  (segment (start 43.4 28.6) (end 43.4 31.8) (width 0.2) (layer "F.Cu") (net 21))
+  (segment (start 43.095 28.295) (end 43.4 28.6) (width 0.2) (layer "F.Cu") (net 21))
+  (segment (start 38.2 37.9) (end 38.2 38.7) (width 0.2) (layer "F.Cu") (net 21))
+  (segment (start 42.2 28.295) (end 43.095 28.295) (width 0.2) (layer "F.Cu") (net 21))
+  (segment (start 43.4 31.8) (end 43.095 32.105) (width 0.2) (layer "F.Cu") (net 21))
+  (segment (start 38.2 34.6) (end 38.2 38.7) (width 0.2) (layer "F.Cu") (net 21))
+  (via (at 38.2 38.7) (size 0.6) (drill 0.3) (layers "F.Cu" "B.Cu") (net 21))
   (via (at 31.05 41) (size 0.6) (drill 0.3) (layers "F.Cu" "B.Cu") (net 21))
-  (segment (start 38.2 38.6) (end 33.7 38.6) (width 0.2) (layer "B.Cu") (net 21))
+  (segment (start 31.05 40.25) (end 32.275 39.025) (width 0.2) (layer "B.Cu") (net 21))
+  (segment (start 32.275 39.025) (end 32.301543 39.025) (width 0.2) (layer "B.Cu") (net 21))
   (segment (start 31.05 40.25) (end 31.05 41) (width 0.5) (layer "B.Cu") (net 21))
-  (segment (start 31.05 40.05) (end 31.05 40.25) (width 0.2) (layer "B.Cu") (net 21))
-  (segment (start 33 39.3) (end 31.8 39.3) (width 0.2) (layer "B.Cu") (net 21))
-  (segment (start 33.7 38.6) (end 33 39.3) (width 0.2) (layer "B.Cu") (net 21))
-  (segment (start 31.8 39.3) (end 31.05 40.05) (width 0.2) (layer "B.Cu") (net 21))
+  (segment (start 32.301543 39.025) (end 32.53 38.796543) (width 0.2) (layer "B.Cu") (net 21))
+  (segment (start 32.6 38.7) (end 38.2 38.7) (width 0.2) (layer "B.Cu") (net 21))
+  (segment (start 32.53 38.796543) (end 32.53 38.77) (width 0.2) (layer "B.Cu") (net 21))
+  (segment (start 32.53 38.77) (end 32.6 38.7) (width 0.2) (layer "B.Cu") (net 21))
   (segment (start 42.2 30.835) (end 40.735 30.835) (width 0.2) (layer "F.Cu") (net 22))
-  (segment (start 33.25 40.8) (end 33.25 39.05) (width 0.5) (layer "F.Cu") (net 22))
-  (segment (start 32.95 37.7) (end 32.95 38.7) (width 0.2) (layer "F.Cu") (net 22))
-  (segment (start 32.95 41) (end 33.05 41) (width 0.2) (layer "F.Cu") (net 22))
-  (segment (start 33.05 41) (end 33.25 40.8) (width 0.2) (layer "F.Cu") (net 22))
   (segment (start 40.735 30.835) (end 40.7 30.8) (width 0.2) (layer "F.Cu") (net 22))
   (segment (start 40.7 30.8) (end 39.8 30.8) (width 0.2) (layer "F.Cu") (net 22))
   (segment (start 36.4 34.2) (end 36.4 40.3) (width 0.2) (layer "F.Cu") (net 22))
+  (segment (start 36.4 40.2) (end 36.4 37.9) (width 0.2) (layer "F.Cu") (net 22))
   (segment (start 41.035 29.565) (end 40.7 29.9) (width 0.2) (layer "F.Cu") (net 22))
-  (segment (start 32.95 38.7) (end 33.25 39) (width 0.2) (layer "F.Cu") (net 22))
   (segment (start 42.2 29.565) (end 41.035 29.565) (width 0.2) (layer "F.Cu") (net 22))
   (segment (start 40.7 29.9) (end 40.7 30.8) (width 0.2) (layer "F.Cu") (net 22))
@@
   (via (at 32.95 41) (size 0.6) (drill 0.3) (layers "F.Cu" "B.Cu") (net 22))
   (segment (start 32.95 41) (end 32.95 40.3) (width 0.5) (layer "B.Cu") (net 22))
-  (segment (start 32.9 40.3) (end 32.95 40.25) (width 0.5) (layer "B.Cu") (net 22))
   (segment (start 36.35 40.25) (end 32.95 40.25) (width 0.2) (layer "B.Cu") (net 22))
   (segment (start 32.95 41) (end 32.95 40.25) (width 0.2) (layer "B.Cu") (net 22))

Commit message: Added PWREN pullup and moved LED 5V to switched
Parts:
- added R5: 10K, Medo64:R (0805), B.Cu at (21.9, 32.5)
Connections:
- R2 pad 1: 5V -> 5V_SW
- R3 pad 1: 5V -> 5V_SW
Routing:
- net 5V_SW: track 24.1 -> 56.9 mm, vias 2 -> 3
- net 5V: track 53.4 -> 27.6 mm
- net PWREN#: track 11.6 -> 16.7 mm
- net GND: track 67.7 -> 72.3 mm
- net LED_TXD: track 32.7 -> 32.0 mm
Other:
- board text added: "Rs485IsoFEC B"
- board text removed: "Rs485IsoFEC A"

Commit message: Aligned resistors
Parts:
- moved C4 1.50 mm to (24.8, 32.5)
Routing:
- net PWREN#: track 16.7 -> 18.2 mm
- net 5V: track 27.6 -> 29.0 mm
- net 5V_SW: track 56.9 -> 56.4 mm
Changed lines of the file:
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@@
   )
   (footprint "Medo64:C (0805)" (layer "B.Cu")
-    (at 24.8 31 90)
+    (at 24.8 32.5 90)
     (tags "CAPC2013X140N")
     (attr smd)
@@
   (via (at 27.4 30.1) (size 0.6) (drill 0.3) (layers "F.Cu" "B.Cu") (net 3))
   (via (at 24.15 29.4) (size 0.6) (drill 0.3) (layers "F.Cu" "B.Cu") (net 3))
-  (segment (start 24.8 30.1) (end 24.9 30.1) (width 0.2) (layer "B.Cu") (net 3))
-  (segment (start 25.6 29.4) (end 24.9 30.1) (width 0.2) (layer "B.Cu") (net 3))
-  (segment (start 24.9 30.1) (end 25.6 30.8) (width 0.2) (layer "B.Cu") (net 3))
+  (segment (start 21.9 31.55) (end 22.05 31.55) (width 0.2) (layer "B.Cu") (net 3))
   (segment (start 33.1 28) (end 33.1 30.1) (width 0.2) (layer "B.Cu") (net 3))
   (segment (start 28.7 30.1) (end 27.4 30.1) (width 0.2) (layer "B.Cu") (net 3))
-  (segment (start 24.8 30.1) (end 24.15 29.45) (width 0.2) (layer "B.Cu") (net 3))
+  (segment (start 25.6 30.8) (end 24.8 31.6) (width 0.2) (layer "B.Cu") (net 3))
   (segment (start 33.1 30.1) (end 28.7 30.1) (width 0.2) (layer "B.Cu") (net 3))
+  (segment (start 26.7 29.4) (end 24.8 29.4) (width 0.2) (layer "B.Cu") (net 3))
   (segment (start 27.4 30.1) (end 26.7 29.4) (width 0.2) (layer "B.Cu") (net 3))
   (segment (start 33.35 31.15) (end 33.35 30.35) (width 0.2) (layer "B.Cu") (net 3))
+  (segment (start 24.8 29.4) (end 24.15 29.4) (width 0.2) (layer "B.Cu") (net 3))
   (segment (start 28.7 29.1) (end 28.7 27.95) (width 0.2) (layer "B.Cu") (net 3))
+  (segment (start 24.8 31.6) (end 24.8 29.4) (width 0.2) (layer "B.Cu") (net 3))
   (segment (start 28.7 30.1) (end 28.7 29.1) (width 0.2) (layer "B.Cu") (net 3))
   (segment (start 24.15 29.45) (end 24.15 29.4) (width 0.2) (layer "B.Cu") (net 3))
-  (segment (start 23.5 30.1) (end 24.8 30.1) (width 0.2) (layer "B.Cu") (net 3))
-  (segment (start 21.9 31.55) (end 22.05 31.55) (width 0.2) (layer "B.Cu") (net 3))
-  (segment (start 22.05 31.55) (end 23.5 30.1) (width 0.2) (layer "B.Cu") (net 3))
-  (segment (start 26.7 29.4) (end 25.6 29.4) (width 0.2) (layer "B.Cu") (net 3))
+  (segment (start 22.05 31.55) (end 24.15 29.45) (width 0.2) (layer "B.Cu") (net 3))
   (segment (start 33.35 30.35) (end 33.1 30.1) (width 0.2) (layer "B.Cu") (net 3))
   (segment (start 31.45 28.45) (end 31.705 28.195) (width 0.2) (layer "F.Cu") (net 4))
@@
   (via (at 39.7 30.1) (size 0.6) (drill 0.3) (layers "F.Cu" "B.Cu") (net 7))
   (via (at 34.245 34.645) (size 0.6) (drill 0.3) (layers "F.Cu" "B.Cu") (net 7))
-  (segment (start 20.8 32.1) (end 20.8 30.1) (width 0.2) (layer "B.Cu") (net 7))
-  (segment (start 21.9 29) (end 21.9 28.05) (width 0.2) (layer "B.Cu") (net 7))
+  (segment (start 21.3 32.6) (end 20.8 32.1) (width 0.2) (layer "B.Cu") (net 7))
   (segment (start 30.9 27.175) (end 31.925 27.175) (width 0.2) (layer "B.Cu") (net 7))
-  (segment (start 22.7 32.6) (end 21.3 32.6) (width 0.2) (layer "B.Cu") (net 7))
   (segment (start 24.4 28.3) (end 24.15 28.05) (width 0.2) (layer "B.Cu") (net 7))
-  (segment (start 21.3 32.6) (end 20.8 32.1) (width 0.2) (layer "B.Cu") (net 7))
-  (segment (start 23.4 31.9) (end 22.7 32.6) (width 0.2) (layer "B.Cu") (net 7))
   (segment (start 34.75 22.1) (end 34.75 23.05) (width 0.2) (layer "B.Cu") (net 7))
   (segment (start 34.6 24.3) (end 34.6 23.2) (width 0.2) (layer "B.Cu") (net 7))
   (segment (start 35.3 34.8) (end 37.5 34.8) (width 0.2) (layer "B.Cu") (net 7))
-  (segment (start 24.8 31.9) (end 23.4 31.9) (width 0.2) (layer "B.Cu") (net 7))
   (segment (start 28.4 24.2) (end 25.9 24.2) (width 0.2) (layer "B.Cu") (net 7))
   (segment (start 29.4 23.2) (end 28.4 24.2) (width 0.2) (layer "B.Cu") (net 7))
@@
   (segment (start 35.3 24.5) (end 35.3 26.2) (width 0.2) (layer "B.Cu") (net 7))
   (segment (start 29.25 23.05) (end 29.25 22.1) (width 0.2) (layer "B.Cu") (net 7))
-  (segment (start 20.8 30.1) (end 21.9 29) (width 0.2) (layer "B.Cu") (net 7))
+  (segment (start 24.8 33.4) (end 23.5 33.4) (width 0.2) (layer "B.Cu") (net 7))
+  (segment (start 22.7 32.6) (end 21.3 32.6) (width 0.2) (layer "B.Cu") (net 7))
   (segment (start 24.15 28.05) (end 23.9 28.05) (width 0.2) (layer "B.Cu") (net 7))
   (segment (start 33.4 24.3) (end 34.5 24.3) (width 0.2) (layer "B.Cu") (net 7))
   (segment (start 25.625 27.175) (end 27.3 27.175) (width 0.2) (layer "B.Cu") (net 7))
   (segment (start 35.1 24.3) (end 35.3 24.5) (width 0.2) (layer "B.Cu") (net 7))
+  (segment (start 21.9 29) (end 21.9 28.05) (width 0.2) (layer "B.Cu") (net 7))
   (segment (start 37.5 26.2) (end 35.3 26.2) (width 0.2) (layer "B.Cu") (net 7))
   (segment (start 31.925 27.175) (end 32.9 26.2) (width 0.2) (layer "B.Cu") (net 7))
@@
   (segment (start 29.4 23.2) (end 29.25 23.05) (width 0.2) (layer "B.Cu") (net 7))
   (segment (start 34.75 23.05) (end 34.6 23.2) (width 0.2) (layer "B.Cu") (net 7))
+  (segment (start 20.8 32.1) (end 20.8 30.1) (width 0.2) (layer "B.Cu") (net 7))
   (segment (start 27.3 27.175) (end 30.9 27.175) (width 0.2) (layer "B.Cu") (net 7))
   (segment (start 33.1 26.2) (end 33.1 24.6) (width 0.2) (layer "B.Cu") (net 7))
   (segment (start 30.9 29) (end 30.9 28) (width 0.2) (layer "B.Cu") (net 7))
   (segment (start 24.8 28) (end 25.625 27.175) (width 0.2) (layer "B.Cu") (net 7))
+  (segment (start 23.5 33.4) (end 22.7 32.6) (width 0.2) (layer "B.Cu") (net 7))
+  (segment (start 20.8 30.1) (end 21.9 29) (width 0.2) (layer "B.Cu") (net 7))
   (segment (start 34.5 24.3) (end 34.6 24.3) (width 0.2) (layer "B.Cu") (net 7))
   (segment (start 34.245 34.645) (end 34.845 34.645) (width 0.2) (layer "B.Cu") (net 7))
@@
   (via (at 25 42.7) (size 0.6) (drill 0.3) (layers "F.Cu" "B.Cu") (net 14))
   (via (at 35.3 28.9) (size 0.6) (drill 0.3) (layers "F.Cu" "B.Cu") (net 14))
+  (segment (start 27.3 34.2) (end 26.8 34.7) (width 0.2) (layer "B.Cu") (net 14))
+  (segment (start 27.3 34.2) (end 30.325 34.2) (width 0.2) (layer "B.Cu") (net 14))
   (segment (start 37.5 28) (end 35.3 28) (width 0.2) (layer "B.Cu") (net 14))
-  (segment (start 23.7 38.854265) (end 23.7 42.7) (width 0.2) (layer "B.Cu") (net 14))
+  (segment (start 23.000001 35.899999) (end 23.000001 38.154266) (width 0.2) (layer "B.Cu") (net 14))
+  (segment (start 24.2 34.7) (end 23.000001 35.899999) (width 0.2) (layer "B.Cu") (net 14))
   (segment (start 22.65 43.05) (end 22.65 44.1) (width 0.2) (layer "B.Cu") (net 14))
-  (segment (start 24.2 34.2) (end 22.7 35.7) (width 0.2) (layer "B.Cu") (net 14))
   (segment (start 39.45 44.1) (end 39.45 43.05) (width 0.2) (layer "B.Cu") (net 14))
-  (segment (start 27.3 34.2) (end 24.2 34.2) (width 0.2) (layer "B.Cu") (net 14))
   (segment (start 27.3 33.2) (end 27.3 34.2) (width 0.2) (layer "B.Cu") (net 14))
+  (segment (start 26.8 34.7) (end 24.2 34.7) (width 0.2) (layer "B.Cu") (net 14))
   (segment (start 35.3 33.3) (end 34.35 33.3) (width 0.2) (layer "B.Cu") (net 14))
   (segment (start 35.3 33.1) (end 35.3 28) (width 0.2) (layer "B.Cu") (net 14))
+  (segment (start 23.7 38.854265) (end 23.7 42.7) (width 0.2) (layer "B.Cu") (net 14))
   (segment (start 34.275 33.2) (end 32.65 33.2) (width 0.2) (layer "B.Cu") (net 14))
-  (segment (start 23.000001 38.154266) (end 23.7 38.854265) (width 0.2) (layer "B.Cu") (net 14))
-  (segment (start 22.7 37.807704) (end 22.880304 37.993882) (width 0.2) (layer "B.Cu") (net 14))
-  (segment (start 30.325 34.2) (end 31.075 33.45) (width 0.2) (layer "B.Cu") (net 14))
   (segment (start 38.799659 42.399659) (end 25.300341 42.399659) (width 0.2) (layer "B.Cu") (net 14))
   (segment (start 25.300341 42.399659) (end 25 42.7) (width 0.2) (layer "B.Cu") (net 14))
   (segment (start 25 42.7) (end 23.7 42.7) (width 0.2) (layer "B.Cu") (net 14))
   (segment (start 35.3 28.9) (end 35.3 28) (width 0.2) (layer "B.Cu") (net 14))
-  (segment (start 27.3 34.2) (end 30.325 34.2) (width 0.2) (layer "B.Cu") (net 14))
-  (segment (start 22.880304 37.993882) (end 23.000001 38.154266) (width 0.2) (layer "B.Cu") (net 14))
   (segment (start 23.7 42.7) (end 23 42.7) (width 0.2) (layer "B.Cu") (net 14))
   (segment (start 23 42.7) (end 22.65 43.05) (width 0.2) (layer "B.Cu") (net 14))
+  (segment (start 30.325 34.2) (end 31.075 33.45) (width 0.2) (layer "B.Cu") (net 14))
   (segment (start 31.075 33.45) (end 32.4 33.45) (width 0.2) (layer "B.Cu") (net 14))
-  (segment (start 22.7 35.7) (end 22.7 37.807704) (width 0.2) (layer "B.Cu") (net 14))
+  (segment (start 23.000001 38.154266) (end 23.7 38.854265) (width 0.2) (layer "B.Cu") (net 14))
   (segment (start 35.3 33) (end 37.5 33) (width 0.2) (layer "B.Cu") (net 14))
   (segment (start 39.45 43.05) (end 38.799659 42.399659) (width 0.2) (layer "B.Cu") (net 14))
@@
   (via (at 26.263909 30.1) (size 0.6) (drill 0.3) (layers "F.Cu" "B.Cu") (net 16))
   (segment (start 28.9 33.45) (end 28.9 32.8) (width 0.2) (layer "B.Cu") (net 16))
-  (segment (start 26.2 32.375) (end 25.125 33.45) (width 0.2) (layer "B.Cu") (net 16))
   (segment (start 26.2 30.163909) (end 26.263909 30.1) (width 0.2) (layer "B.Cu") (net 16))
   (segment (start 28.9 32.8) (end 28.475 32.375) (width 0.2) (layer "B.Cu") (net 16))
+  (segment (start 25.7 34.3) (end 22.75 34.3) (width 0.2) (layer "B.Cu") (net 16))
   (segment (start 26.2 32.375) (end 26.2 30.163909) (width 0.2) (layer "B.Cu") (net 16))
+  (segment (start 26.2 33.8) (end 25.7 34.3) (width 0.2) (layer "B.Cu") (net 16))
+  (segment (start 26.2 32.375) (end 26.2 33.8) (width 0.2) (layer "B.Cu") (net 16))
+  (segment (start 22.75 34.3) (end 21.9 33.45) (width 0.2) (layer "B.Cu") (net 16))
   (segment (start 28.475 32.375) (end 26.2 32.375) (width 0.2) (layer "B.Cu") (net 16))
-  (segment (start 25.125 33.45) (end 21.9 33.45) (width 0.2) (layer "B.Cu") (net 16))
   (segment (start 29.1 26.425) (end 30.375 26.425) (width 0.2) (layer "F.Cu") (net 17))
   (segment (start 34.25 27.95) (end 34.25 29.55) (width 0.2) (layer "F.Cu") (net 17))
